File: Eagle/JX1/Main Board/Main Board.sch (EAGLE design)
At the start: 16 parts, among them U1 SN74HC595N, U2 SN74HC595N

Commit message: Worked on heater traces some more.
Connections:
- net +12V: now also BED_HEAT-2.KL, E_HEAT-1.KL
Other:
- moved on the sheet: BED_HEAT-1, BED_HEAT-2, E_HEAT-2
Changed lines of the file:
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@@
 <part name="BED_THERM" library="con-wago-500" library_urn="urn:adsk.eagle:library:195" deviceset="W237-102" device="" package3d_urn="urn:adsk.eagle:package:10688/1"/>
 <part name="E_THERM" library="con-wago-500" library_urn="urn:adsk.eagle:library:195" deviceset="W237-102" device="" package3d_urn="urn:adsk.eagle:package:10688/1"/>
+<part name="P+10" library="supply1" library_urn="urn:adsk.eagle:library:371" deviceset="+12V" device=""/>
 </parts>
 <sheets>
@@
 <attribute name="VALUE" x="78.74" y="7.62" size="1.778" layer="96"/>
 </instance>
-<instance part="BED_HEAT" gate="-1" x="48.26" y="58.42" smashed="yes">
-<attribute name="NAME" x="48.26" y="59.309" size="1.778" layer="95" rot="R180"/>
-</instance>
-<instance part="BED_HEAT" gate="-2" x="48.26" y="53.34" smashed="yes">
-<attribute name="VALUE" x="45.72" y="49.657" size="1.778" layer="96"/>
-<attribute name="NAME" x="48.26" y="54.229" size="1.778" layer="95" rot="R180"/>
+<instance part="BED_HEAT" gate="-1" x="45.72" y="55.88" smashed="yes">
+<attribute name="NAME" x="45.72" y="56.769" size="1.778" layer="95" rot="R180"/>
+</instance>
+<instance part="BED_HEAT" gate="-2" x="17.78" y="43.18" smashed="yes">
+<attribute name="VALUE" x="15.24" y="39.497" size="1.778" layer="96"/>
+<attribute name="NAME" x="17.78" y="44.069" size="1.778" layer="95" rot="R180"/>
 </instance>
 <instance part="E_HEAT" gate="-1" x="38.1" y="43.18" smashed="yes" rot="R180">
 <attribute name="NAME" x="38.1" y="42.291" size="1.778" layer="95"/>
 </instance>
-<instance part="E_HEAT" gate="-2" x="38.1" y="48.26" smashed="yes" rot="R180">
-<attribute name="VALUE" x="40.64" y="51.943" size="1.778" layer="96" rot="R180"/>
-<attribute name="NAME" x="38.1" y="47.371" size="1.778" layer="95"/>
+<instance part="E_HEAT" gate="-2" x="48.26" y="50.8" smashed="yes" rot="R180">
+<attribute name="VALUE" x="50.8" y="54.483" size="1.778" layer="96" rot="R180"/>
+<attribute name="NAME" x="48.26" y="49.911" size="1.778" layer="95"/>
 </instance>
 <instance part="GND7" gate="1" x="71.12" y="58.42" smashed="yes">
@@
 <attribute name="VALUE" x="15.24" y="74.803" size="1.778" layer="96" rot="R180"/>
 <attribute name="NAME" x="12.7" y="70.231" size="1.778" layer="95"/>
+</instance>
+<instance part="P+10" gate="1" x="27.94" y="45.72" smashed="yes">
+<attribute name="VALUE" x="35.306" y="46.482" size="1.778" layer="96" rot="R180"/>
 </instance>
 </instances>
@@
 <pinref part="P+3" gate="1" pin="+12V"/>
 </segment>
+<segment>
+<pinref part="E_HEAT" gate="-1" pin="KL"/>
+<pinref part="P+10" gate="1" pin="+12V"/>
+<wire x1="33.02" y1="43.18" x2="27.94" y2="43.18" width="0.1524" layer="91"/>
+<pinref part="BED_HEAT" gate="-2" pin="KL"/>
+<wire x1="22.86" y1="43.18" x2="27.94" y2="43.18" width="0.1524" layer="91"/>
+<junction x="27.94" y="43.18"/>
+</segment>
 </net>

Commit message: Started added power mosfets for heaters
Parts:
- added Q1, Q2: IRF3704L-V, transistor-power:IRF3704L-V
- added R3, R4: 1k, eagle-ltspice:R0207/10
Connections:
- new net N$4: E_HEAT-2.KL, Q1.D
- new net N$5: Q2.G, R3.2
- new net N$6: BED_HEAT-1.KL, Q2.D
- new net N$7: Q1.G, R4.2
- new net N$8: R4.1
- new net N$9: R3.1
- net GND: now also Q1.S, Q2.S
Other:
- moved on the sheet: B1, B2, B3, B4, BED_HEAT-1, BED_HEAT-2, BED_THERM-1, BED_THERM-2, E_HEAT-1, E_HEAT-2, E_THERM-1, E_THERM-2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
